File: uart-friend2-usb/uart-friend2-usb.kicad_sch (KiCad schematic)
At the start: 42 parts, among them J1 USB_C_Receptacle_USB2.0, P1 USB_A_Plug_PCB, P2 USB_C_Plug_USB2.0_16P, P3 USB_C_Plug_USB2.0_16P, P4 USB_C_Plug_USB3.0_9P, SW1 BOOT, SW2 RST, U1 RP2040, U2 W25Q128JVPIQ, U3 NCP1117-3.3_SOT223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

Commit message: resolve uart-friend2-usb footprint issues
Parts:
- removed U3: NCP1117-3.3_SOT223, Package_TO_SOT_SMD:SOT-223-3_TabPin2, symbol Regulator_Linear:NCP1117-3.3_SOT223
- added C16: 0.1uF, Capacitor_SMD:C_0402_1005Metric, symbol Device:C_Small
- added D3, D4: Green, LED_SMD:LED_0402_1005Metric, symbol Device:LED_Small_Filled
- added J2: Conn_02x03_Odd_Even, uart-friend2-usb-special:TC2030-NL_SMALL, symbol Connector_Generic:Conn_02x03_Odd_Even
- added R10, R11, R12, R13, R14, R9: 5.1k, Resistor_SMD:R_0402_1005Metric, symbol Device:R_Small
- added R8: 1k, Resistor_SMD:R_0402_1005Metric, symbol Device:R_Small
- added U4: AP7366-33W5-7, Package_TO_SOT_SMD:SOT-23-5, symbol uart-friend2-usb:AP7366-33W5-7
- J1: footprint Connector_USB:USB_C_Receptacle_GCT_USB4135-GF-A_6P_TopMnt_Horizontal -> Connector_USB:USB_C_Receptacle_G-Switch_GT-USB-7010ASV; Mfg SHOU HAN -> G-Switch; Mfg PN TYPE-C-6P-073 -> GT-USB-7010ASV
- P1: footprint uart-friend2-usb-special:USB_A_Plug_PCB_SparkFun -> uart-friend2-usb-special:USB_A_Plug_PCB_Shorter_Pads
- SW1, SW2: footprint (none) -> Button_Switch_SMD:SW_SPST_FSMSM; Mfg (none) -> BZCN; Mfg PN (none) -> TSB008A2530A03; Mfg2 (none) -> Panasonic; Mfg2 PN (none) -> FSMSM
- U1: symbol MCU_RaspberryPi:RP2040 -> uart-friend2-usb:RP2040_not_hidden
Connections:
- net +3V3: now also J2.1 (Pin_1), U4.5 (OUT)
- net GND: now also C16.2, D3.1 (K), D4.1 (K), J2.5 (Pin_5), R10.2, R11.1, R12.1, R9.2, U4.2 (GND)
- net SWD: now also J2.2 (Pin_2); no longer TP3.1
- net SWD_CLK: now also J2.4 (Pin_4); no longer TP2.1
- net U1_RUN: now also C16.1, R8.1
- net USB0_R_N: no longer P2.B7 (D-)
- net USB0_R_P: no longer P2.B6 (D+)
- net USB1_N: now also R5.1, U1.3 (GPIO1); no longer J1.A7 (D-), J1.B7 (D-), P3.A7 (D-), P3.B7 (D-), R5.2
- net USB1_P: now also R6.1, U1.2 (GPIO0); no longer J1.A6 (D+), J1.B6 (D+), P3.A6 (D+), P3.B6 (D+), R6.2
- net VBUS: now also U4.1 (IN), U4.3 (EN)
- net VBUS0: now also P4.A4 (VBUS), P4.A9 (VBUS), P4.B4 (VBUS), P4.B9 (VBUS)
- net at P2.A5 (CC): now also R11.2
- net J1_CC1: now reaches J1.A5 (CC1)
- net J1_CC1: now also R9.1
- net J2_CC2: now reaches J1.B5 (CC2)
- net J2_CC2: now also R10.1
- net ADC1: now reaches TP1.1
- net ADC1: now also U1.39 (GPIO27_ADC1)
- net P4_CC: now reaches P4.A5 (CC)
- net P4_CC: now also R12.2
- net LED_GPIO8: now reaches U1.11 (GPIO8)
- net LED_GPIO8: now also R13.1
- net ADC2: now reaches U1.40 (GPIO28_ADC2)
- net ADC2: now also TP2.1
- net LED_GPIO7: now reaches U1.9 (GPIO7)
- net LED_GPIO7: now also R14.1
- new net: D4.2 (A), R14.2
- new net: D3.2 (A), R13.2
- new net SWD_OUT: J2.6 (Pin_6), TP3.1
- new net SWD_RST: J2.3 (Pin_3), R8.2
- new net USB1_R_N: J1.A7 (D-), J1.B7 (D-), P3.A7 (D-), R5.2
- new net USB1_R_P: J1.A6 (D+), J1.B6 (D+), P3.A6 (D+), R6.2
- no-connect marks 6 -> 10
Other:
- note added: "C1/1uF for VREG_IN/44 0.1uF per set of adjacent IOVDD/AVDD pins"
- note added: "C9/1uF for VREG_VOUT/45 0.1uF per DVDD pin"
- note removed: "C1/1uF for VREG_IN on 44 0.1uF per IOVDD/AVDD"
- note removed: "C9/1uF for VREG_VOUT on 45 0.1uF per DVDD"
- moved on the sheet: TP2, TP3

Commit message: uart-friend2-usb floorplan and some layout
Parts:
- removed C8: 0.1uF, Capacitor_SMD:C_0402_1005Metric, symbol Device:C_Small
- added D5, D6: Green, LED_SMD:LED_0402_1005Metric, symbol Device:LED_Small_Filled
- added R15, R16: 5.1k, Resistor_SMD:R_0402_1005Metric, symbol Device:R_Small
- added U3, U5: WE-TVS-82400102, Package_TO_SOT_SMD:SOT-23-6, symbol Power_Protection:WE-TVS-82400102
- C12, C13: value 4.7uF -> 2.2uF; footprint Capacitor_SMD:C_0805_2012Metric -> Capacitor_SMD:C_0603_1608Metric
- D3, D4: value Green -> Orange
Connections:
- net GND: now also P1.4 (GND), D5.1 (K), D6.1 (K), U3.2, U5.2; no longer P1.A1 (GND), P1.A12 (GND), P1.B1 (GND), P1.B12 (GND)
- net USB0_R_N: now also U3.3; no longer P1.A7 (D-), P2.A7 (D-), P4.A7 (D-)
- net USB0_R_P: now also U3.1; no longer P1.A6 (D+), P2.A6 (D+), P4.A6 (D+)
- net USB1_R_N: now also U5.1; no longer J1.A7 (D-), J1.B7 (D-), P3.A7 (D-)
- net USB1_R_P: now also U5.3; no longer J1.A6 (D+), J1.B6 (D+), P3.A6 (D+)
- net VBUS0: now also P1.1 (VBUS), R15.1, U3.5; no longer P1.A4 (VBUS), P1.A9 (VBUS), P1.B4 (VBUS), P1.B9 (VBUS)
- net VBUS1: now also R16.1, U5.5
- new net: D5.2 (A), R15.2
- new net: D6.2 (A), R16.2
- new net USB0_D_N: P1.2 (D-), P2.A7 (D-), P4.A7 (D-), U3.4
- new net USB0_D_P: P1.3 (D+), P2.A6 (D+), P4.A6 (D+), U3.6
- new net USB1_D_N: J1.A7 (D-), J1.B7 (D-), P3.A7 (D-), U5.6
- new net USB1_D_P: J1.A6 (D+), J1.B6 (D+), P3.A6 (D+), U5.4
Other:
- note added: "Native USB Side One connector to be used at a time; J2 or J3 populated."
- note added: "PIO USB Side One connector to be used at a time."
- note added: "Place close to J1/P3"
- note added: "Place close to P1/P2/P4"
- note added: "Place close to U1"
- note removed: "Native USB Side Singular use; J2 or J3 populated."
- note removed: "PIO USB Side Singular use."
- moved on the sheet: R1, R2
